File: pcb/BarsaPad kicad.kicad_pcb (KiCad board)
At the start: 2 copper layers, 62 x 50 mm, 13 parts, among them J1 Conn_01x04, SW1 SW_Push, SW2 SW_Push, SW3 SW_Push, U1 MOUDLE-SEEEDUINO-XIAO

Commit message: updated
Parts:
- removed REF** (x4): MountingHole_3.2mm_M3, MountingHole:MountingHole_3.2mm_M3
- moved J1 11.5 mm to (57.5, 10.5)
- moved ENC1 4.75 mm to (3.75, 11.6)
Routing:
- net Net-(J1-Pin_4): track 32.3 -> 43.8 mm
- net Net-(J1-Pin_3): track 32.5 -> 44.0 mm
- net +3.3V: track 32.8 -> 44.3 mm, vias 0 -> 1
- net Net-(U1-PB08_A6_D6_TX): track 87.0 -> 91.8 mm
- net Net-(U1-PB09_A7_D7_RX): track 36.8 -> 41.5 mm
- net Net-(U1-PA7_A8_D8_SCK): track 28.7 -> 33.4 mm
